Commit message: Reused STL files and aligned the model with the axis

File: dpr4_description/urdf/dpr4_description_old.urdf (robot description, URDF)
Before this commit: robot dpr4_description, 7 links, 6 joints
Links:
- link AandrijfwielLinks: geometry collision mesh filename=package://dpr4_description/meshes/AandrijfwielLinks.STL; visual mesh filename=package://dpr4_description/meshes/AandrijfwielLinks.STL
- link AandrijfwielRechts: geometry collision mesh filename=package://dpr4_description/meshes/AandrijfwielRechts.STL; visual mesh filename=package://dpr4_description/meshes/AandrijfwielRechts.STL
- link PassiefLinkLinks: geometry collision mesh filename=package://dpr4_description/meshes/PassiefLinkLinks.STL; visual mesh filename=package://dpr4_description/meshes/PassiefLinkLinks.STL
- link PassiefLinkRechts: geometry collision mesh filename=package://dpr4_description/meshes/PassiefLinkRechts.STL; visual mesh filename=package://dpr4_description/meshes/PassiefLinkRechts.STL
- link ZwenkwielLinks: geometry collision mesh filename=package://dpr4_description/meshes/ZwenkwielLinks.STL; visual mesh filename=package://dpr4_description/meshes/ZwenkwielLinks.STL
- link ZwenkwielRechts: geometry collision mesh filename=package://dpr4_description/meshes/ZwenkwielRechts.STL; visual mesh filename=package://dpr4_description/meshes/ZwenkwielRechts.STL
- link base_link: mass 12.0 -> 11.846925821453; geometry collision mesh filename=package://dpr4_description/meshes/base_link.STL; visual mesh filename=package://dpr4_description/meshes/base_link.STL
Joints:
- joint AandrijfwielJointLinks: origin xyz=-0.272 0.084 0.145 rpy=0 0 0 -> xyz=-0.0282464240706431 -0.268065095057138 0.156065936359952 rpy=0.833624618439072 1.33733009515224E-15 1.42420629036135
- joint AandrijfwielJointRechts: origin xyz=0.272 0.084 0.145 rpy=0 0 0 -> xyz=0.0450645120366924 0.228456132827706 0.156065936359953 rpy=1.45340093763758 2.27107070527088E-16 1.42420629036135
- joint PassiefJointLinks: origin xyz=-0.183 0.532 0.182 rpy=0 0 0 -> xyz=0.426071935947264 -0.258167122222898 0.0780659363599518 rpy=1.5707963267949 -8.97790964757775E-18 -0.147155764293911
- joint PassiefJointRechts: origin xyz=0.183 0.532 0.182 rpy=0 0 0 -> xyz=0.479531944388918 0.103907493702353 0.0780659363599517 rpy=1.5707963267949 -9.23902259508227E-18 -0.151468187968226
- joint ZwenkwielJointLinks: origin xyz=0 0.04025 -0.105 rpy=0 0 0 -> xyz=0.0402530425707102 0.0100000000000001 0 rpy=1.57759894294971 1.57079630572147 -0.799615214926937
- joint ZwenkwielJointRechts: origin xyz=0 0.04025 -0.105 rpy=0 0 0 -> xyz=0.0402530425707104 0.0100000000000002 0 rpy=0.788698481447936 1.57079631189374 -0.363147009946176
