Commit message: Fixed center of mass

File: dpr4_description/urdf/dpr4_description.urdf (robot description, URDF)
Before this commit: robot dpr4_description, 7 links, 6 joints
Joints:
- joint PassiefJointLinks: axis 0 1 0 -> 0 0 1
- joint PassiefJointRechts: axis 0 1 0 -> 0 0 1

Commit message: Translated and improved names of files/links/joints

File: dpr4_description/urdf/dpr4_description.urdf (robot description, URDF)
Before this commit: robot dpr4_description, 7 links, 6 joints
Links:
- removed link AandrijfwielLinks
- removed link AandrijfwielRechts
- removed link PassiefLinkLinks
- removed link PassiefLinkRechts
- removed link ZwenkwielLinks
- removed link ZwenkwielRechts
- added link back_wheel_left, mass 0.2926460297435; collision mesh filename=package://dpr4_description/meshes/back_wheel.stl; visual mesh filename=package://dpr4_description/meshes/back_wheel.stl
- added link back_wheel_right, mass 0.29264656535805; collision mesh filename=package://dpr4_description/meshes/back_wheel.stl; visual mesh filename=package://dpr4_description/meshes/back_wheel.stl
- added link front_wheel_left, mass 1.98850951394841; collision mesh filename=package://dpr4_description/meshes/front_wheel.stl; visual mesh filename=package://dpr4_description/meshes/front_wheel.stl
- added link front_wheel_right, mass 1.98850951394841; collision mesh filename=package://dpr4_description/meshes/front_wheel.stl; visual mesh filename=package://dpr4_description/meshes/front_wheel.stl
- added link yoke_left, mass 0.027578120885064; collision mesh filename=package://dpr4_description/meshes/yoke.stl; visual mesh filename=package://dpr4_description/meshes/yoke.stl
- added link yoke_right, mass 0.0275781208850642; collision mesh filename=package://dpr4_description/meshes/yoke.stl; visual mesh filename=package://dpr4_description/meshes/yoke.stl
Joints:
- removed joint AandrijfwielJointLinks
- removed joint AandrijfwielJointRechts
- removed joint PassiefJointLinks
- removed joint PassiefJointRechts
- removed joint ZwenkwielJointLinks
- removed joint ZwenkwielJointRechts
- added joint back_wheel_left_joint: type continuous, parent yoke_left, child back_wheel_left, origin xyz=0 0.04025 -0.105 rpy=0 0 0, axis -1 0 0
- added joint back_wheel_right_joint: type continuous, parent yoke_right, child back_wheel_right, origin xyz=0 0.04025 -0.105 rpy=0 0 0, axis -1 0 0
- added joint front_wheel_left_joint: type continuous, parent base_link, child front_wheel_left, origin xyz=-0.272 0.084 0.145 rpy=0 0 0, axis -1 0 0
- added joint front_wheel_right_joint: type continuous, parent base_link, child front_wheel_right, origin xyz=0.272 0.084 0.145 rpy=0 0 0, axis -1 0 0
- added joint yoke_left_joint: type continuous, parent base_link, child yoke_left, origin xyz=-0.183 0.532 0.182 rpy=0 0 0, axis 0 0 1
- added joint yoke_right_joint: type continuous, parent base_link, child yoke_right, origin xyz=0.183 0.532 0.182 rpy=0 0 0, axis 0 0 1
