Commit message: Converted the urdf file to a xacro file

File: urdf/dpr4_description.urdf.xacro (robot description, xacro)
@@ -1,4 +1,4 @@
 <?xml version="1.0" encoding="UTF-8"?>
-<robot name="dpr4_description">
+<robot name="dpr4_description" xmlns:xacro="http://ros.org/wiki/xacro">
   <!-- Colors -->
   <gazebo reference="front_wheel_left">
@@ -59,5 +59,4 @@
         <mesh filename="package://dpr4_description/meshes/front_wheel.stl" />
       </geometry>
-      <material name=""> Gazebo/Blue </material>
     </visual>
     <collision>
@@ -96,5 +95,5 @@
       <origin xyz="0 0.01701 -0.04258" rpy="0 0 0" />
       <mass value="0.027578120885064" />
-      <inertia ixx="0.00004501" ixy="0.0000000000000000" ixz="0.0000000000000000" iyy="0.00004508" iyz="-0.00001339" izz="0.00002122" />
+      <inertia ixx="0.0000770000000000" ixy="0.0000000000000000" ixz="0.0000000000000000" iyy="0.0000750000000000" iyz="-0.000000000000000" izz="0.0000260000000000" />
     </inertial>
     <visual>
@@ -119,5 +118,5 @@
       <origin xyz="0 0.01701 -0.04258" rpy="0 0 0" />
       <mass value="0.0275781208850642" />
-      <inertia ixx="0.0000770000000000" ixy="0.0000000000000000" ixz="0.0000000000000000" iyy="0.0000750000000000" iyz="-0.0000250000000000" izz="0.0000260000000000" />
+      <inertia ixx="0.0000770000000000" ixy="0.0000000000000000" ixz="0.0000000000000000" iyy="0.0000750000000000" iyz="-0.000000000000000" izz="0.0000260000000000" />
     </inertial>
     <visual>

Commit message: Changed Inertia Tensor of Base_link

File: urdf/dpr4_description.urdf.xacro (robot description, xacro)
@@ -29,5 +29,5 @@
       <origin xyz="0 0.23146 0.14798" rpy="0 0 0" />
       <mass value="12.0" />
-      <inertia ixx="1.30161345" ixy="-0.00690756" ixz="-0.00131153" iyy="0.47311975" iyz="0.47495754" izz="1.25649724" />
+      <inertia ixx="0.3625" ixy="0" ixz="0" iyy="0.1625" iyz="0" izz="0.52" />
     </inertial>
     <visual>

Commit message: Introduce subsampled collision geometry.
And update the xacro to make use of them.

File: urdf/dpr4_description.urdf.xacro (robot description, xacro)
@@ -34,5 +34,5 @@
       <origin xyz="0 0 0" rpy="0 0 0" />
       <geometry>
-        <mesh filename="package://dpr4_description/meshes/base_link.stl" />
+        <mesh filename="package://dpr4_description/meshes/visual/base_link.stl" />
       </geometry>
       <material name="">
@@ -43,5 +43,5 @@
       <origin xyz="0 0 0" rpy="0 0 0" />
       <geometry>
-        <mesh filename="package://dpr4_description/meshes/base_link.stl" />
+        <mesh filename="package://dpr4_description/meshes/collision/base_link.stl" />
       </geometry>
     </collision>
@@ -57,11 +57,11 @@
       <origin xyz="0 0 0" rpy="0 0 0" />
       <geometry>
-        <mesh filename="package://dpr4_description/meshes/front_wheel.stl" />
-      </geometry>
-    </visual>
-    <collision>
-      <origin xyz="0 0 0" rpy="0 0 0" />
-      <geometry>
-        <mesh filename="package://dpr4_description/meshes/front_wheel.stl" />
+        <mesh filename="package://dpr4_description/meshes/visual/front_wheel.stl" />
+      </geometry>
+    </visual>
+    <collision>
+      <origin xyz="0 0 0" rpy="0 0 0" />
+      <geometry>
+        <mesh filename="package://dpr4_description/meshes/collision/front_wheel.stl" />
       </geometry>
     </collision>
@@ -77,5 +77,5 @@
       <origin xyz="0 0 0" rpy="0 0 0" />
       <geometry>
-        <mesh filename="package://dpr4_description/meshes/front_wheel.stl" />
+        <mesh filename="package://dpr4_description/meshes/visual/front_wheel.stl" />
       </geometry>
       <material name="">
@@ -86,5 +86,5 @@
       <origin xyz="0 0 0" rpy="0 0 0" />
       <geometry>
-        <mesh filename="package://dpr4_description/meshes/front_wheel.stl" />
+        <mesh filename="package://dpr4_description/meshes/collision/front_wheel.stl" />
       </geometry>
     </collision>
@@ -100,5 +100,5 @@
       <origin xyz="0 0 0" rpy="0 0 0" />
       <geometry>
-        <mesh filename="package://dpr4_description/meshes/yoke.stl" />
+        <mesh filename="package://dpr4_description/meshes/visual/yoke.stl" />
       </geometry>
       <material name="">
@@ -109,5 +109,5 @@
       <origin xyz="0 0 0" rpy="0 0 0" />
       <geometry>
-        <mesh filename="package://dpr4_description/meshes/yoke.stl" />
+        <mesh filename="package://dpr4_description/meshes/collision/yoke.stl" />
       </geometry>
     </collision>
@@ -123,5 +123,5 @@
       <origin xyz="0 0 0" rpy="0 0 0" />
       <geometry>
-        <mesh filename="package://dpr4_description/meshes/yoke.stl" />
+        <mesh filename="package://dpr4_description/meshes/visual/yoke.stl" />
       </geometry>
       <material name="">
@@ -132,5 +132,5 @@
       <origin xyz="0 0 0" rpy="0 0 0" />
       <geometry>
-        <mesh filename="package://dpr4_description/meshes/yoke.stl" />
+        <mesh filename="package://dpr4_description/meshes/collision/yoke.stl" />
       </geometry>
     </collision>
@@ -146,5 +146,5 @@
       <origin xyz="0 0 0" rpy="0 0 0" />
       <geometry>
-        <mesh filename="package://dpr4_description/meshes/back_wheel.stl" />
+        <mesh filename="package://dpr4_description/meshes/visual/back_wheel.stl" />
       </geometry>
       <material name="">
@@ -155,5 +155,5 @@
       <origin xyz="0 0 0" rpy="0 0 0" />
       <geometry>
-        <mesh filename="package://dpr4_description/meshes/back_wheel.stl" />
+        <mesh filename="package://dpr4_description/meshes/collision/back_wheel.stl" />
       </geometry>
     </collision>
@@ -169,5 +169,5 @@
       <origin xyz="0 0 0" rpy="0 0 0" />
       <geometry>
-        <mesh filename="package://dpr4_description/meshes/back_wheel.stl" />
+        <mesh filename="package://dpr4_description/meshes/visual/back_wheel.stl" />
       </geometry>
       <material name="">
@@ -178,5 +178,5 @@
       <origin xyz="0 0 0" rpy="0 0 0" />
       <geometry>
-        <mesh filename="package://dpr4_description/meshes/back_wheel.stl" />
+        <mesh filename="package://dpr4_description/meshes/collision/back_wheel.stl" />
       </geometry>
     </collision>

Commit message: Added xacro macro for the front wheels

File: urdf/dpr4_description.urdf.xacro (robot description, xacro)
@@ -1,4 +1,7 @@
 <?xml version="1.0" encoding="UTF-8"?>
 <robot name="dpr4_description" xmlns:xacro="http://ros.org/wiki/xacro">
+  <xacro:include filename="$(find dpr4_description)/urdf/front_wheel.urdf.xacro" />
+  <!-- <xacro:include filename="$(find dpr4_description)/urdf/back_wheel.urdf.xacro" />
+  <xacro:include filename="$(find dpr4_description)/urdf/yokes.urdf.xacro"/> -->
   <!-- Colors -->
   <gazebo reference="front_wheel_left">
@@ -48,46 +51,6 @@
   </link>
   <!-- The big wheel on front, used to move the robot -->
-  <link name="front_wheel_left">
-    <inertial>
-      <origin xyz="0 0 0" rpy="0 0 0" />
-      <mass value="1.98850951394841" />
-      <inertia ixx="0.0254040000000000" ixy="0.0000000000000000" ixz="0.0000000000000000" iyy="0.0130220000000000" iyz="0.0000000000000000" izz="0.0130220000000000" />
-    </inertial>
-    <visual>
-      <origin xyz="0 0 0" rpy="0 0 0" />
-      <geometry>
-        <mesh filename="package://dpr4_description/meshes/visual/front_wheel.stl" />
-      </geometry>
-    </visual>
-    <collision>
-      <origin xyz="0 0 0" rpy="0 0 0" />
-      <geometry>
-        <mesh filename="package://dpr4_description/meshes/collision/front_wheel.stl" />
-      </geometry>
-    </collision>
-  </link>
-  <!-- The big wheel on front, used to move the robot -->
-  <link name="front_wheel_right">
-    <inertial>
-      <origin xyz="0 0 0" rpy="0 0 0" />
-      <mass value="1.98850951394841" />
-      <inertia ixx="0.0254040000000000" ixy="0.0000000000000000" ixz="0.0000000000000000" iyy="0.0130220000000000" iyz="0.0000000000000000" izz="0.0130220000000000" />
-    </inertial>
-    <visual>
-      <origin xyz="0 0 0" rpy="0 0 0" />
-      <geometry>
-        <mesh filename="package://dpr4_description/meshes/visual/front_wheel.stl" />
-      </geometry>
-      <material name="">
-        <color rgba="0.294117647058824 0.294117647058824 0.294117647058824 1" />
-      </material>
-    </visual>
-    <collision>
-      <origin xyz="0 0 0" rpy="0 0 0" />
-      <geometry>
-        <mesh filename="package://dpr4_description/meshes/collision/front_wheel.stl" />
-      </geometry>
-    </collision>
-  </link>
+  <xacro:front_wheel parent="base_link" name="front_wheel_left" x_loc="-0.272" y_loc="0.084" z_loc="0.145"/>
+  <xacro:front_wheel parent="base_link" name="front_wheel_right" x_loc="0.272" y_loc="0.084" z_loc="0.145"/>
   <!-- The part connecting the back wheel to the base -->
   <link name="yoke_left">
@@ -183,16 +146,4 @@
   </link>
   <!-- The joints -->
-  <joint name="front_wheel_left_joint" type="continuous">
-    <origin xyz="-0.272 0.084 0.145" rpy="0 0 0" />
-    <parent link="base_link" />
-    <child link="front_wheel_left" />
-    <axis xyz="-1 0 0" />
-  </joint>
-  <joint name="front_wheel_right_joint" type="continuous">
-    <origin xyz="0.272 0.084 0.145" rpy="0 0 0" />
-    <parent link="base_link" />
-    <child link="front_wheel_right" />
-    <axis xyz="-1 0 0" />
-  </joint>
   <joint name="yoke_left_joint" type="continuous">
     <origin xyz="-0.183 0.532 0.182" rpy="0 0 0" />

Commit message: Added xacro macro for yoke

File: urdf/dpr4_description.urdf.xacro (robot description, xacro)
@@ -2,6 +2,6 @@
 <robot name="dpr4_description" xmlns:xacro="http://ros.org/wiki/xacro">
   <xacro:include filename="$(find dpr4_description)/urdf/front_wheel.urdf.xacro" />
-  <!-- <xacro:include filename="$(find dpr4_description)/urdf/back_wheel.urdf.xacro" />
-  <xacro:include filename="$(find dpr4_description)/urdf/yokes.urdf.xacro"/> -->
+  <!-- <xacro:include filename="$(find dpr4_description)/urdf/back_wheel.urdf.xacro" /> -->
+  <xacro:include filename="$(find dpr4_description)/urdf/yoke.urdf.xacro"/>
   <!-- Colors -->
   <gazebo reference="front_wheel_left">
@@ -50,54 +50,11 @@
     </collision>
   </link>
-  <!-- The big wheel on front, used to move the robot -->
+  <!-- The big wheels on front, used to move the robot -->
   <xacro:front_wheel parent="base_link" name="front_wheel_left" x_loc="-0.272" y_loc="0.084" z_loc="0.145"/>
   <xacro:front_wheel parent="base_link" name="front_wheel_right" x_loc="0.272" y_loc="0.084" z_loc="0.145"/>
-  <!-- The part connecting the back wheel to the base -->
-  <link name="yoke_left">
-    <inertial>
-      <origin xyz="0 0.01701 -0.04258" rpy="0 0 0" />
-      <mass value="0.027578120885064" />
-      <inertia ixx="0.0000770000000000" ixy="0.0000000000000000" ixz="0.0000000000000000" iyy="0.0000750000000000" iyz="-0.000000000000000" izz="0.0000260000000000" />
-    </inertial>
-    <visual>
-      <origin xyz="0 0 0" rpy="0 0 0" />
-      <geometry>
-        <mesh filename="package://dpr4_description/meshes/visual/yoke.stl" />
-      </geometry>
-      <material name="">
-        <color rgba="0.752941176470588 0.752941176470588 0.752941176470588 1" />
-      </material>
-    </visual>
-    <collision>
-      <origin xyz="0 0 0" rpy="0 0 0" />
-      <geometry>
-        <mesh filename="package://dpr4_description/meshes/collision/yoke.stl" />
-      </geometry>
-    </collision>
-  </link>
-  <!-- The part connecting the back wheel to the base -->
-  <link name="yoke_right">
-    <inertial>
-      <origin xyz="0 0.01701 -0.04258" rpy="0 0 0" />
-      <mass value="0.0275781208850642" />
-      <inertia ixx="0.0000770000000000" ixy="0.0000000000000000" ixz="0.0000000000000000" iyy="0.0000750000000000" iyz="-0.000000000000000" izz="0.0000260000000000" />
-    </inertial>
-    <visual>
-      <origin xyz="0 0 0" rpy="0 0 0" />
-      <geometry>
-        <mesh filename="package://dpr4_description/meshes/visual/yoke.stl" />
-      </geometry>
-      <material name="">
-        <color rgba="0.752941176470588 0.752941176470588 0.752941176470588 1" />
-      </material>
-    </visual>
-    <collision>
-      <origin xyz="0 0 0" rpy="0 0 0" />
-      <geometry>
-        <mesh filename="package://dpr4_description/meshes/collision/yoke.stl" />
-      </geometry>
-    </collision>
-  </link>
-  <!-- The small wheel on the back -->
+  <!-- The parts connecting the back wheel to the base -->
+  <xacro:yoke parent="base_link" name="yoke_left" x_loc="-0.183" y_loc="0.532" z_loc="0.182"/>
+  <xacro:yoke parent="base_link" name="yoke_right" x_loc="0.183" y_loc="0.532" z_loc="0.182"/>
+  <!-- The small wheels on the back -->
   <link name="back_wheel_left">
     <inertial>
@@ -146,19 +103,7 @@
   </link>
   <!-- The joints -->
-  <joint name="yoke_left_joint" type="continuous">
-    <origin xyz="-0.183 0.532 0.182" rpy="0 0 0" />
-    <parent link="base_link" />
-    <child link="yoke_left" />
-    <axis xyz="0 0 1" />
-  </joint>
-  <joint name="yoke_right_joint" type="continuous">
-    <origin xyz="0.183 0.532 0.182" rpy="0 0 0" />
-    <parent link="base_link" />
-    <child link="yoke_right" />
-    <axis xyz="0 0 1" />
-  </joint>
   <joint name="back_wheel_left_joint" type="continuous">
     <origin xyz="0 0.04025 -0.105" rpy="0 0 0" />
-    <parent link="yoke_left" />
+    <parent link="yoke_left_link" />
     <child link="back_wheel_left" />
     <axis xyz="-1 0 0" />
@@ -166,5 +111,5 @@
   <joint name="back_wheel_right_joint" type="continuous">
     <origin xyz="0 0.04025 -0.105" rpy="0 0 0" />
-    <parent link="yoke_right" />
+    <parent link="yoke_right_link" />
     <child link="back_wheel_right" />
     <axis xyz="-1 0 0" />

Commit message: Added xacro macro for the back wheels

File: urdf/dpr4_description.urdf.xacro (robot description, xacro)
@@ -2,5 +2,5 @@
 <robot name="dpr4_description" xmlns:xacro="http://ros.org/wiki/xacro">
   <xacro:include filename="$(find dpr4_description)/urdf/front_wheel.urdf.xacro" />
-  <!-- <xacro:include filename="$(find dpr4_description)/urdf/back_wheel.urdf.xacro" /> -->
+  <xacro:include filename="$(find dpr4_description)/urdf/back_wheel.urdf.xacro" />
   <xacro:include filename="$(find dpr4_description)/urdf/yoke.urdf.xacro"/>
   <!-- Colors -->
@@ -57,61 +57,6 @@
   <xacro:yoke parent="base_link" name="yoke_right" x_loc="0.183" y_loc="0.532" z_loc="0.182"/>
   <!-- The small wheels on the back -->
-  <link name="back_wheel_left">
-    <inertial>
-      <origin xyz="0 0 0" rpy="0 0 0" />
-      <mass value="0.2926460297435" />
-      <inertia ixx="0.0009700000000000" ixy="0.0000000000000000" ixz="0.0000000000000000" iyy="0.0005000000000000" iyz="0.0000000000000000" izz="0.0005000000000000" />
-    </inertial>
-    <visual>
-      <origin xyz="0 0 0" rpy="0 0 0" />
-      <geometry>
-        <mesh filename="package://dpr4_description/meshes/visual/back_wheel.stl" />
-      </geometry>
-      <material name="">
-        <color rgba="0.294117647058824 0.294117647058824 0.294117647058824 1" />
-      </material>
-    </visual>
-    <collision>
-      <origin xyz="0 0 0" rpy="0 0 0" />
-      <geometry>
-        <mesh filename="package://dpr4_description/meshes/collision/back_wheel.stl" />
-      </geometry>
-    </collision>
-  </link>
-  <!-- The small wheel on the back -->
-  <link name="back_wheel_right">
-    <inertial>
-      <origin xyz="0 0 0" rpy="0 0 0" />
-      <mass value="0.29264656535805" />
-      <inertia ixx="0.0009700000000000" ixy="0.0000000000000000" ixz="0.0000000000000000" iyy="0.0005000000000000" iyz="0.0000000000000000" izz="0.0005000000000000" />
-    </inertial>
-    <visual>
-      <origin xyz="0 0 0" rpy="0 0 0" />
-      <geometry>
-        <mesh filename="package://dpr4_description/meshes/visual/back_wheel.stl" />
-      </geometry>
-      <material name="">
-        <color rgba="0.294117647058824 0.294117647058824 0.294117647058824 1" />
-      </material>
-    </visual>
-    <collision>
-      <origin xyz="0 0 0" rpy="0 0 0" />
-      <geometry>
-        <mesh filename="package://dpr4_description/meshes/collision/back_wheel.stl" />
-      </geometry>
-    </collision>
-  </link>
+  <xacro:back_wheel parent="yoke_left_link" name="back_wheel_left" x_loc="0" y_loc="0.04025" z_loc="-0.105"/>
+  <xacro:back_wheel parent="yoke_right_link" name="back_wheel_right" x_loc="0" y_loc="0.04025" z_loc="-0.105"/>
   <!-- The joints -->
-  <joint name="back_wheel_left_joint" type="continuous">
-    <origin xyz="0 0.04025 -0.105" rpy="0 0 0" />
-    <parent link="yoke_left_link" />
-    <child link="back_wheel_left" />
-    <axis xyz="-1 0 0" />
-  </joint>
-  <joint name="back_wheel_right_joint" type="continuous">
-    <origin xyz="0 0.04025 -0.105" rpy="0 0 0" />
-    <parent link="yoke_right_link" />
-    <child link="back_wheel_right" />
-    <axis xyz="-1 0 0" />
-  </joint>
 </robot>

Commit message: Made the whole dpr4 a macro

File: urdf/dpr4_description.urdf.xacro (robot description, xacro)
@@ -1,4 +1,5 @@
 <?xml version="1.0" encoding="UTF-8"?>
 <robot name="dpr4_description" xmlns:xacro="http://ros.org/wiki/xacro">
+<xacro:macro name="dpr4" params="name">
   <xacro:include filename="$(find dpr4_description)/urdf/front_wheel.urdf.xacro" />
   <xacro:include filename="$(find dpr4_description)/urdf/back_wheel.urdf.xacro" />
@@ -28,5 +29,5 @@
   <!-- Links -->
   <!-- Main part of the base. -->
-  <link name="base_link">
+  <link name="${name}">
     <inertial>
       <origin xyz="0 0.23146 0.14798" rpy="0 0 0" />
@@ -59,4 +60,4 @@
   <xacro:back_wheel parent="yoke_left_link" name="back_wheel_left" x_loc="0" y_loc="0.04025" z_loc="-0.105"/>
   <xacro:back_wheel parent="yoke_right_link" name="back_wheel_right" x_loc="0" y_loc="0.04025" z_loc="-0.105"/>
-  <!-- The joints -->
+</xacro:macro>
 </robot>
