Commit message: Rotated base to make it point towards the postive x axis

File: urdf/back_wheel.urdf.xacro (robot description, xacro)
@@ -1,7 +1,7 @@
 <?xml version="1.0"?>
 <robot name="dpr4_back_wheel" xmlns:xacro="http://ros.org/wiki/xacro">
-<xacro:macro name="back_wheel" params="parent name x_loc y_loc z_loc">
+<xacro:macro name="back_wheel" params="parent name *joint_origin">
 <joint name="${name}_link" type="continuous">
-  <origin xyz="${x_loc} ${y_loc} ${z_loc}" rpy="0 0 0" />
+  <xacro:insert_block name="joint_origin" />
   <parent link="${parent}" />
   <child link="${name}_link" />

File: urdf/dpr4_description.urdf.xacro (robot description, xacro)
@@ -31,10 +31,10 @@
   <link name="${name}">
     <inertial>
-      <origin xyz="0 0.23146 0.14798" rpy="0 0 0" />
+      <origin xyz="-0.23146 0 0.14798" rpy="0 0 0" />
       <mass value="12.0" />
-      <inertia ixx="0.3625" ixy="0" ixz="0" iyy="0.1625" iyz="0" izz="0.52" />
+      <inertia iyy="0.3625" ixy="0" ixz="0" ixx="0.1625" iyz="0" izz="0.52" />
     </inertial>
     <visual>
-      <origin xyz="0 0 0" rpy="0 0 0" />
+      <origin xyz="0 0 0" rpy="0 0 1.57" />
       <geometry>
         <mesh filename="package://dpr4_description/meshes/visual/base_link.stl" />
@@ -45,5 +45,5 @@
     </visual>
     <collision>
-      <origin xyz="0 0 0" rpy="0 0 0" />
+      <origin xyz="0 0 0" rpy="0 0 1.57" />
       <geometry>
         <mesh filename="package://dpr4_description/meshes/collision/base_link.stl" />
@@ -52,12 +52,24 @@
   </link>
   <!-- The big wheels on front, used to move the robot -->
-  <xacro:front_wheel parent="base_link" name="front_wheel_left" x_loc="-0.272" y_loc="0.084" z_loc="0.145"/>
-  <xacro:front_wheel parent="base_link" name="front_wheel_right" x_loc="0.272" y_loc="0.084" z_loc="0.145"/>
+  <xacro:front_wheel parent="${name}" name="front_wheel_left">
+    <origin xyz="-0.084 -0.272 0.145" rpy="0 0 -1.57" />
+  </xacro:front_wheel>
+  <xacro:front_wheel parent="${name}" name="front_wheel_right">
+    <origin xyz="-0.084 0.272 0.145" rpy="0 0 -1.57" />
+  </xacro:front_wheel>
   <!-- The parts connecting the back wheel to the base -->
-  <xacro:yoke parent="base_link" name="yoke_left" x_loc="-0.183" y_loc="0.532" z_loc="0.182"/>
-  <xacro:yoke parent="base_link" name="yoke_right" x_loc="0.183" y_loc="0.532" z_loc="0.182"/>
+  <xacro:yoke parent="${name}" name="yoke_left" >
+    <origin xyz="-0.532 -0.183 0.182" rpy="0 0 -1.57" />
+  </xacro:yoke>
+  <xacro:yoke parent="${name}" name="yoke_right" >
+    <origin xyz="-0.532 0.183 0.182" rpy="0 0 -1.57" />
+  </xacro:yoke>
   <!-- The small wheels on the back -->
-  <xacro:back_wheel parent="yoke_left_link" name="back_wheel_left" x_loc="0" y_loc="0.04025" z_loc="-0.105"/>
-  <xacro:back_wheel parent="yoke_right_link" name="back_wheel_right" x_loc="0" y_loc="0.04025" z_loc="-0.105"/>
+  <xacro:back_wheel parent="yoke_left_link" name="back_wheel_left" >
+    <origin xyz="0 0.04025 -0.105" rpy="0 0 0" />
+  </xacro:back_wheel>
+  <xacro:back_wheel parent="yoke_right_link" name="back_wheel_right" >
+    <origin xyz="0 0.04025 -0.105" rpy="0 0 0" />
+  </xacro:back_wheel>
 </xacro:macro>
 </robot>

File: urdf/front_wheel.urdf.xacro (robot description, xacro)
@@ -1,7 +1,7 @@
 <?xml version="1.0"?>
 <robot name="dpr4_front_wheel" xmlns:xacro="http://ros.org/wiki/xacro">
-<xacro:macro name="front_wheel" params="parent name x_loc y_loc z_loc">
+<xacro:macro name="front_wheel" params="parent name *joint_origin">
 <joint name="${name}_joint" type="continuous">
-  <origin xyz="${x_loc} ${y_loc} ${z_loc}" rpy="0 0 0" />
+  <xacro:insert_block name="joint_origin" />
   <parent link="${parent}" />
   <child link="${name}_link" />

File: urdf/yoke.urdf.xacro (robot description, xacro)
@@ -1,7 +1,7 @@
 <?xml version="1.0"?>
 <robot name="dpr4_yoke" xmlns:xacro="http://ros.org/wiki/xacro">
-<xacro:macro name="yoke" params="parent name x_loc y_loc z_loc">
+<xacro:macro name="yoke" params="parent name *joint_origin">
 <joint name="${name}_link" type="continuous">
-  <origin xyz="${x_loc} ${y_loc} ${z_loc}" rpy="0 0 0" />
+  <xacro:insert_block name="joint_origin" />
   <parent link="${parent}" />
   <child link="${name}_link" />
